File: pcb/hopper.kicad_sch (KiCad schematic)
At the start: 29 parts, among them J1 AudioJack2, J2 AudioJack2, J3 AudioJack2, J4 AudioJack2, J5 DIN-5_180degree, J6 DIN-5_180degree, J7 Conn_01x02_Pin, K1 G5V-2, K2 G5V-2, SW1 SW_Push, SW2 SW_Push, SW3 SW_Push, SW4 SW_SP3T, SW5 SW_SP3T, SW6 SW_SP3T, SW7 SW_SP3T, SW8 SW_SP3T, SW9 SW_SP3T, U1 STM32H745IITx, U2 CS4272, U3 6N139

Commit message: stuff
Parts:
- added C1, C2: C, symbol Device:C
- added C10, C11, C12, C13, C14, C15, C17, C18, C19, C20, C21, C22, C23, C24, C25, C26, C27, C29, C3, C33, C5, C6, C7, C8, C9: 100n, symbol Device:C
- added C16: 4.7u, symbol Device:C_Polarized
- added C28, C32, C4: 1u, symbol Device:C_Polarized
- added C30, C31: 0.2u, symbol Device:C
- added J8: SWD, symbol Connector_Generic:Conn_02x05_Odd_Even
- added L1: L, symbol Device:L
- added R1, R3: 10k, symbol Device:R
- added R2: 0, symbol Device:R
- added SW10: Reset, symbol Switch:SW_Push
- added SW11: Boot, symbol Switch:SW_Push_SPDT
- added Y1: Crystal_GND23, symbol Device:Crystal_GND23
Connections:
- net GND: now also U1.100 (VSS), U1.106 (VSS), U1.112 (VSS), U1.119 (VSS), U1.12 (VSS), U1.134 (VSS), U1.137 (VSS), U1.14 (VSSSMPS), U1.15 (VLXSMPS), U1.151 (VSS), U1.159 (VSS), U1.16 (VDDSMPS), U1.17 (VFBSMPS), U1.173 (VSS), U1.24 (VSS), U1.38 (VSSA), U1.45 (VSS), U1.47 (VSS), U1.6 (VSS), U1.64 (VSS), U1.70 (VSS), U1.81 (VSS), U1.83 (VSS), U1.93 (VSS), C1.2, C10.2, C11.2, C12.2, C13.2, C14.2, C15.2, C16.2, C17.2, C18.2, C19.2, C2.2, C20.2, C21.2, C22.2, C23.2, C24.2, C25.2, C26.2, C27.2, C28.2, C29.2, C3.2, C30.2, C31.2, C32.2, C33.2, C4.2, C5.2, C6.2, C7.2, C8.2, C9.2, J8.3 (Pin_3), J8.5 (Pin_5), SW10.1, SW11.1 (A), Y1.2, Y1.3
- net VDD: now reaches U1.105 (VDD)
- net VDD: now also U1.113 (VDD), U1.120 (VDD50_USB), U1.121 (VDD33_USB), U1.126 (VDD), U1.13 (VDD), U1.135 (VDDLDO), U1.136 (VDD), U1.152 (VDD), U1.160 (VDD), U1.175 (VDDLDO), U1.176 (VDD), U1.25 (VDD), U1.44 (VDD), U1.48 (VDD), U1.65 (VDD), U1.7 (VDD), U1.71 (VDD), U1.8 (VBAT), U1.82 (VDDLDO), U1.84 (VDD), U1.92 (VDD), U1.99 (VDD), C10.1, C11.1, C12.1, C13.1, C14.1, C15.1, C16.1, C17.1, C18.1, C19.1, C20.1, C21.1, C22.1, C23.1, C24.1, C25.1, C26.1, C27.1, C32.1, C33.1, C6.1, C7.1, C8.1, C9.1, L1.1
- net SWDIO: now reaches U1.132 (PA13)
- net SWDIO: now also J8.2 (Pin_2)
- net at U1.133 (VCAP): now also U1.172 (VCAP), U1.80 (VCAP), C30.1, C31.1
- net SWCLK: now reaches U1.138 (PA14)
- net SWCLK: now also J8.4 (Pin_4)
- net SWO: now reaches U1.162 (PB3)
- net SWO: now also J8.6 (Pin_6)
- net BOOT: now reaches U1.167 (BOOT0)
- net BOOT: now also R1.2
- net at U1.174 (PDR_ON): now also R3.1
- net CRYSTAL1: now reaches U1.31 (PH0)
- net CRYSTAL1: now also C1.1, Y1.1
- net CRYSTAL2: now reaches U1.32 (PH1)
- net CRYSTAL2: now also C2.1, Y1.4
- net RST: now reaches U1.33 (NRST)
- net RST: now also C3.1, J8.10 (Pin_10), SW10.2
- net VREF+: now reaches U1.39 (VREF+)
- net VREF+: now also C28.1, C29.1, R2.1
- net VDDA: now reaches U1.40 (VDDA)
- net VDDA: now also C4.1, C5.1, L1.2, R2.2
- new net: R1.1, SW11.2 (B)
- new net +3.3V: J8.1 (Pin_1), R3.2, SW11.3 (C)
- no-connect marks 0 -> 3
Other:
- note added: "Ceramic low esr"
- note added: "Near usb power pins"
- moved on the sheet: J1, J2, J3, J4, J5, J6, J7, K1, K2, RV1, RV2, RV3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

Commit message: stuff
Parts:
- added C34: 100u, symbol Device:C_Polarized
- added C35, C39, C59: 100n, symbol Device:C
- added C36, C37: 220n, symbol Device:C
- added C38, C52, C53, C60, C61: 10u, symbol Device:C_Polarized
- added C40, C49, C55, C56, C63, C64: 470p, symbol Device:C
- added C41, C50: 1.5n, symbol Device:C
- added C42, C46: 2200p, symbol Device:C
- added C43, C47: 6.8n, symbol Device:C
- added C44, C45, C48, C51: 22u, symbol Device:C_Polarized
- added C54, C62: 10n, symbol Device:C
- added C57, C65: 2700p, symbol Device:C
- added C58: 1u, symbol Device:C_Polarized
- added D1: D_Schottky, symbol Device:D_Schottky
- added R10, R11, R19, R27: 47k, symbol Device:R
- added R12, R20: 4.42k, symbol Device:R
- added R13, R21: 1.33k, symbol Device:R
- added R14, R22: 2.32k, symbol Device:R
- added R15, R23: 715r, symbol Device:R
- added R16, R25: 4.99k, symbol Device:R
- added R17, R24: 1.5k, symbol Device:R
- added R18, R26: 560r, symbol Device:R
- added R28, R29, R34, R35, R6, R8: 10k, symbol Device:R
- added R30, R33, R36, R38: 634r, symbol Device:R
- added R31, R32, R37, R39: 91r, symbol Device:R
- added R4, R5: 1M, symbol Device:R
- added R7, R9: 30.1k, symbol Device:R
- added SW12: Inst/line, symbol Switch:SW_DPDT_x2
- added U4, U5, U6, U7, U8, U9: Opamp_Dual, symbol Device:Opamp_Dual
- J1: value AudioJack2 -> L/mono in
- J2: value AudioJack2 -> R in
Connections:
- net +9V: now also C34.1, C35.1, D1.2 (A)
- net GND: now also J1.S, J2.S, C34.2, C35.2, C38.2, C39.2, C42.1, C43.1, C46.1, C47.1, C54.2, C58.2, C59.2, C62.2, R11.1, R19.1, R27.1, R6.1, R8.1, U4.4 (V-), U5.4 (V-), U6.4 (V-), U7.4 (V-), U8.4 (V-)
- net at J2.T: now also C37.1
- net at J1.T: now also C36.1
- net VCOM: now reaches U2.15 (VCOM)
- net VCOM: now also C54.1, C58.1, C59.1, C62.1, R28.1, R29.2, R34.1, R35.2
- net LIN-: now reaches U2.16 (AINA-)
- net LIN-: now also C57.2, R30.1, R31.1
- net LIN+: now reaches U2.17 (AINA+)
- net LIN+: now also C57.1, R32.1, R33.1
- net RIN+: now reaches U2.18 (AINB+)
- net RIN+: now also C65.1, R36.1, R37.1
- net RIN-: now reaches U2.19 (AINB-)
- net RIN-: now also C65.2, R38.1, R39.1
- net LOUT-: now reaches U2.24 (AOUTA-)
- net LOUT-: now also R12.2
- net LOUT+: now reaches U2.25 (AOUTA+)
- net LOUT+: now also R13.2
- net ROUT+: now reaches U2.26 (AOUTB+)
- net ROUT+: now also R21.2
- net ROUT-: now reaches U2.27 (AOUTB-)
- net ROUT-: now also R20.2
- new net: C61.1, R35.1, U9.5 (+)
- new net: C64.1, R38.2, U9.6 (-)
- new net: C64.2, R39.2, U9.7
- new net: C49.1, R22.1, U7.6 (-)
- new net: C49.2, C51.1, R25.1, U7.7
- new net: C38.1, C39.1, R10.1, R11.2, U6.3 (+)
- new net: C56.1, R33.2, U8.2 (-)
- new net: C56.2, R32.2, U8.1
- new net: C43.2, R13.1, R15.2, R17.2
- new net: C63.2, R37.2, U9.1
- new net: C63.1, R36.2, U9.2 (-)
- new net: C60.1, R34.2, U9.3 (+)
- new net: C52.1, R28.2, U8.3 (+)
- new net: C42.2, R12.1, R14.2, R16.2
- new net: C51.2, R26.2
- new net: C46.2, R20.1, R22.2, R25.2
- new net: C48.1, R24.1
- new net: C47.2, R21.1, R23.2, R24.2
- new net: C50.1, R23.1, U7.5 (+)
- new net: C48.2, C50.2
- new net: R6.2, SW12.2 (B), U4.6 (-)
- new net: C40.1, R14.1, U7.2 (-)
- new net: C40.2, C45.1, R16.1, U7.1
- new net: C41.1, R15.1, U7.3 (+)
- new net: U5.1, U5.2 (-), U5.5 (+)
- new net: C37.2, R5.2, U5.3 (+)
- new net: C44.1, R17.1
- new net: R8.2, SW12.5 (B), U5.6 (-)
- new net: R9.1, SW12.6 (C), U5.7
- new net: C53.1, R29.1, U8.5 (+)
- new net: C55.1, R30.2, U8.6 (-)
- new net: C55.2, R31.2, U8.7
- new net: R9.2, SW12.4 (A)
- new net: C41.2, C44.2
- new net: C45.2, R18.2
- new net: C36.2, R4.2, U4.3 (+)
- new net: R7.2, SW12.1 (A)
- new net: R7.1, SW12.3 (C), U4.7
- new net: U4.1, U4.2 (-), U4.5 (+)
- new net LOUTA: R18.1, R19.2
- new net ROUTA: R26.1, R27.2
- new net VCC: D1.1 (K), R10.2, U4.8 (V+), U5.8 (V+), U6.8 (V+), U7.8 (V+), U8.8 (V+)
- new net VGND: R4.1, R5.1, U6.1, U6.2 (-)
Other:
- moved on the sheet: C10, C11, C12, C13, C14, C15, C16, C17, C18, C19, C20, C21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

Commit message: stuff
Parts:
- removed C52, C53, C60, C61: 10u, symbol Device:C_Polarized
- removed C56, C63, C64: 470p, symbol Device:C
- removed C62: 10n, symbol Device:C
- removed C65: 2700p, symbol Device:C
- removed R35: 10k, symbol Device:R
- removed R36, R38: 634r, symbol Device:R
- removed R37, R39: 91r, symbol Device:R
- removed unit 2 of U8
- removed unit 1 of U8
- removed U9: Opamp_Dual, symbol Device:Opamp_Dual
- added C52, C53, C66: 1n, symbol Device:C
- added R40: 1K, symbol Device:R
- added R41, R42: 40R, symbol Device:R
- added R43, R44: 270R, symbol Device:R
- added U10, U9: OPA1632, symbol emaj:OPA1632
- C54: value 10n -> 2700p
- C55: value 470p -> 1n
- J1: value L/mono in -> L in
- J3: value AudioJack2 -> L out
- J4: value AudioJack2 -> R out
- R1, R3, R6, R8: value 10k -> 10K
- R10, R11, R19, R27: value 47k -> 47K
- R12, R20: value 4.42k -> 4.42K
- R13, R21: value 1.33k -> 1.33K
- R14, R22: value 2.32k -> 2.32K
- R15, R23: value 715r -> 715R
- R16, R25: value 4.99k -> 4.99K
- R17, R24: value 1.5k -> 1.5K
- R18, R26: value 560r -> 560R
- R28, R29: value 10k -> 1K
- R30: value 634r -> 1K
- R31, R32: value 91r -> 270R
- R33: value 634r -> 40R
- R34: value 10k -> 40R
- R7, R9: value 30.1k -> 30.1K
Connections:
- net GND: now also J3.S, J4.S, R30.2, R40.2; no longer C54.2
- net LIN+: now also C57.2, R42.1, R44.1; no longer C57.1, R32.1, R33.1
- net LIN-: now also C57.1, R41.1, R43.1; no longer C57.2, R30.1, R31.1
- net RIN+: now also C54.2, R32.1, R34.1
- net RIN-: now also C54.1, R31.1, R33.1
- net VCOM: now also U10.2 (VOCM), U9.2 (VOCM); no longer C54.1, R28.1, R29.2, R34.1
- net at R33.2: now also C52.2, U9.5 (-)
- net at R32.2: now also R30.1, C53.1, U9.1 (-)
- net at R34.2: now also C53.2, U9.4 (+)
- net at R28.2: now also R7.1, SW12.3 (C), U4.7
- net at K2.11: now also K2.6
- net at K2.13: now also J4.T
- net at K2.4: now also J2.T
- net RIN: now reaches K2.8
- net RIN: now also C37.1
- net ROUT: now reaches K2.9
- net at K1.11: now also K1.6
- net at K1.13: now also J3.T
- net at K1.4: now also J1.T
- net LIN: now reaches K1.8
- net LIN: now also C36.1
- net LOUT: now reaches K1.9
- net at R9.1, SW12.6 (C), U5.7: now also R29.2
- net at R29.1: now also R31.2, C52.1, U9.8 (+)
- net at C55.1: now also R28.1, R43.2, U10.8 (+); no longer R30.2
- net at C55.2: now also R41.2, U10.5 (-); no longer R31.2
- net LOUTA: no longer names the net of R18.1, R19.2
- net ROUTA: no longer names the net of R26.1, R27.2
- new net: C66.1, R40.1, R44.2, U10.1 (-)
- new net: C66.2, R42.2, U10.4 (+)
- new net: U10.6 (V-), U10.9 (V-)
- new net: U9.6 (V-), U9.9 (V-)
Other:
- moved on the sheet: C36, C37, C55, C57, J1, J2, J3, J4, K1, K2, R28, R4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

Commit message: stuff
Parts:
- removed SW11: Boot, symbol Switch:SW_Push_SPDT
- added C56, C60: 10u, symbol Device:C_Polarized
- added R35, R36, R37, R39: 10K, symbol Device:R
- added R38, R45: 100R, symbol Device:R
- added SW11: Boot, symbol Switch:SW_Push
- added SW13: Inst/line out, symbol Switch:SW_DPDT_x2
- added U11: Opamp_Dual, symbol Device:Opamp_Dual
- added unit 2 of U8
- added unit 1 of U8
- SW12: value Inst/line -> Inst/line in
Connections:
- net +3.3V: now also SW11.1
- net BOOT: now also SW11.2
- net GND: now also R1.1, U11.4 (V-); no longer R19.1, R27.1, R6.1, R8.1
- net LOUT: now also C56.2
- net ROUT: now also C60.2
- net VCC: now also U11.8 (V+)
- net VGND: now also R19.1, R27.1, R6.1, R8.1, R35.1, R36.1
- net at R26.1, R27.2: now also U8.5 (+)
- net at R18.1, R19.2: now also U8.3 (+)
- new net: R36.2, SW13.5 (B), U8.6 (-)
- new net: R39.1, R45.2, SW13.4 (A), U8.7
- new net: C56.1, R38.1
- new net: R37.1, R38.2, SW13.1 (A), U8.1
- new net: R37.2, SW13.3 (C)
- new net: C60.1, R45.1
- new net: R35.2, SW13.2 (B), U8.2 (-)
- new net: R39.2, SW13.6 (C)
Other:
- moved on the sheet: C36, C37, C40, C41, C42, C43, C44, C45, C46, C47, C48, C49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

Commit message: stuff
Parts:
- added unit 2 of U7
- added unit 1 of U7
Connections:
- net at C49.1, R22.1: now also U8.2 (-); no longer U7.6 (-)
- net at C49.2, C51.1, R25.1: now also U8.1; no longer U7.7
- net at R37.1, R38.2, SW13.1 (A): now also U7.7; no longer U8.1
- net at C50.1, R23.1: now also U8.3 (+); no longer U7.5 (+)
- net at C40.1, R14.1: now also U7.2 (-); no longer U7.2 (-)
- net at C40.2, C45.1, R16.1: now also U7.1; no longer U7.1
- net at C41.1, R15.1: now also U7.3 (+); no longer U7.3 (+)
- net at R18.1, R19.2: now also U7.5 (+); no longer U8.3 (+)
- net at R35.2, SW13.2 (B): now also U7.6 (-); no longer U8.2 (-)
Other:
- moved on the sheet: U8A
Changed lines of the file:
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@@
 	(symbol
 		(lib_id "Device:Opamp_Dual")
-		(at 237.49 353.06 0)
-		(mirror x)
+		(at 288.29 309.88 0)
 		(unit 2)
 		(exclude_from_sim no)
@@
 		(dnp no)
 		(property "Reference" "U7"
-			(at 245.11 355.092 0)
+			(at 288.036 300.228 0)
 			(effects
 				(font
@@
 		)
 		(property "Value" "Opamp_Dual"
-			(at 248.412 356.87 0)
+			(at 288.29 302.26 0)
 			(effects
 				(font
@@
 		)
 		(property "Footprint" ""
-			(at 237.49 353.06 0)
+			(at 288.29 309.88 0)
 			(effects
 				(font
@@
 		)
 		(property "Datasheet" "~"
-			(at 237.49 353.06 0)
+			(at 288.29 309.88 0)
 			(effects
 				(font
@@
 		)
 		(property "Description" "Dual operational amplifier"
-			(at 237.49 353.06 0)
+			(at 288.29 309.88 0)
 			(effects
 				(font
@@
 		)
 		(property "Sim.Library" "${KICAD9_SYMBOL_DIR}/Simulation_SPICE.sp"
-			(at 237.49 353.06 0)
+			(at 288.29 309.88 0)
 			(effects
 				(font
@@
 		)
 		(property "Sim.Name" "kicad_builtin_opamp_dual"
-			(at 237.49 353.06 0)
+			(at 288.29 309.88 0)
 			(effects
 				(font
@@
 		)
 		(property "Sim.Device" "SUBCKT"
-			(at 237.49 353.06 0)
+			(at 288.29 309.88 0)
 			(effects
 				(font
@@
 		)
 		(property "Sim.Pins" "1=out1 2=in1- 3=in1+ 4=vee 5=in2+ 6=in2- 7=out2 8=vcc"
-			(at 237.49 353.06 0)
+			(at 288.29 309.88 0)
 			(effects
 				(font
@@
 	(symbol
 		(lib_id "Device:Opamp_Dual")
-		(at 288.29 309.88 0)
+		(at 237.49 353.06 0)
+		(mirror x)
 		(unit 1)
 		(exclude_from_sim no)
@@
 		(on_board yes)
 		(dnp no)
-		(fields_autoplaced yes)
 		(property "Reference" "U8"
-			(at 288.29 299.72 0)
+			(at 244.348 354.838 0)
 			(effects
 				(font
@@
 		)
 		(property "Value" "Opamp_Dual"
-			(at 288.29 302.26 0)
+			(at 248.92 356.87 0)
 			(effects
 				(font
@@
 		)
 		(property "Footprint" ""
-			(at 288.29 309.88 0)
+			(at 237.49 353.06 0)
 			(effects
 				(font
@@
 		)
 		(property "Datasheet" "~"
-			(at 288.29 309.88 0)
+			(at 237.49 353.06 0)
 			(effects
 				(font
@@
 		)
 		(property "Description" "Dual operational amplifier"
-			(at 288.29 309.88 0)
+			(at 237.49 353.06 0)
 			(effects
 				(font
@@
 		)
 		(property "Sim.Library" "${KICAD9_SYMBOL_DIR}/Simulation_SPICE.sp"
-			(at 288.29 309.88 0)
+			(at 237.49 353.06 0)
 			(effects
 				(font
@@
 		)
 		(property "Sim.Name" "kicad_builtin_opamp_dual"
-			(at 288.29 309.88 0)
+			(at 237.49 353.06 0)
 			(effects
 				(font
@@
 		)
 		(property "Sim.Device" "SUBCKT"
-			(at 288.29 309.88 0)
+			(at 237.49 353.06 0)
 			(effects
 				(font
@@
 		)
 		(property "Sim.Pins" "1=out1 2=in1- 3=in1+ 4=vee 5=in2+ 6=in2- 7=out2 8=vcc"
-			(at 288.29 309.88 0)
+			(at 237.49 353.06 0)
 			(effects
 				(font

Commit message: stuff
Parts:
- removed C30: 0.2u, symbol Device:C
- removed C40, C49: 470p, symbol Device:C
- removed C41, C50: 1.5n, symbol Device:C
- removed C42, C46: 2200p, symbol Device:C
- removed C43, C47: 6.8n, symbol Device:C
- removed C44, C45, C48, C51: 22u, symbol Device:C_Polarized
- removed C52, C55, C66: 1n, symbol Device:C
- removed C54, C57: 2700p, symbol Device:C
- removed C59: 100n, symbol Device:C
- removed R13: 1.33K, symbol Device:R
- removed R14: 2.32K, symbol Device:R
- removed R15, R23: 715R, symbol Device:R
- removed R16, R25: 4.99K, symbol Device:R
- removed R17, R24: 1.5K, symbol Device:R
- removed R18, R26: 560R, symbol Device:R
- removed R2: 0, symbol Device:R
- removed R27: 47K, symbol Device:R
- removed R28, R29, R30, R40: 1K, symbol Device:R
- removed R31, R32, R43, R44: 270R, symbol Device:R
- removed R33, R34, R41, R42: 40R, symbol Device:R
- removed U10, U9: OPA1632, symbol emaj:OPA1632
- removed U11, U8: Opamp_Dual, symbol Device:Opamp_Dual
- removed U2: CS4272, Package_SO:TSSOP-28_4.4x9.7mm_P0.65mm, symbol Audio:CS4272
- removed unit 1 of U7
- added C10, C11: 4.7u, symbol Device:C_Polarized
- added C14, C17, C19, C27, C38, C7: 100n, symbol Device:C
- added C15, C16, C18, C26, C30, C35, C52: 10u, symbol Device:C_Polarized
- added C47: 22u, symbol Device:C_Polarized
- added C8, C9: 2.2u, symbol Device:C
- added FB1: FerriteBead_Small, symbol Device:FerriteBead_Small
- added R11: 100K, symbol Device:R
- added U4: PCM3060, Package_SO:TSSOP-28_4.4x9.7mm_P0.65mm, symbol Audio:PCM3060
- added unit 2 of U5
- added U7: AMS1117-5.0, Package_TO_SOT_SMD:SOT-223-3_TabPin2, symbol Regulator_Linear:AMS1117-5.0
- added U8: TPS62160DGK, Package_SO:MSOP-8_3x3mm_P0.65mm, symbol Regulator_Switching:TPS62160DGK
- added U9: AMS1117-3.3, Package_TO_SOT_SMD:SOT-223-3_TabPin2, symbol Regulator_Linear:AMS1117-3.3
- C53: value 1n -> 100n
- C58: value 1u -> 10u
- C6: renamed from C31; value 0.2u -> 2.2u
- L1: value L -> 2.2uH
- R12: value 4.42K -> 100K
- R19: value 47K -> 100K
- R20: value 4.42K -> 220K
- R21: value 1.33K -> 100K
- R22: value 2.32K -> 47R
- renumbered C33 to C12, C32 to C13, C36 to C2, C34 to C20, C38 to C21, C35 to C22, C39 to C23, C56 to C24, C60 to C25, C4 to C29, C37 to C3, C29 to C31, C5 to C32, C6 to C33, C17 to C34, C7 to C36, C18 to C37, C8 to C39, C3 to C4, C19 to C40, C9 to C41, C20 to C42, C10 to C43, C21 to C44, C11 to C45, C22 to C46, C12 to C48, C23 to C49, C2 to C5, C13 to C50, C24 to C51, C14 to C54, C25 to C55, C15 to C56, C26 to C57, C16 to C59, C27 to C60, J8 to J1, J7 to J2, J1 to J3, J3 to J4, J2 to J5, J4 to J6, J5 to J7, J6 to J8, R4 to R1, R11 to R10, R35 to R13, R36 to R14, R37 to R15, R39 to R16, R38 to R17, R45 to R18, R5 to R2, R1 to R3, R8 to R4, R6 to R5, R3 to R6, R9 to R8, R10 to R9, SW10 to SW1, SW7 to SW10, SW8 to SW11, SW3 to SW12, SW9 to SW13, SW11 to SW2, SW12 to SW3, SW13 to SW4, SW4 to SW5, SW1 to SW6, SW5 to SW7, SW6 to SW8, SW2 to SW9, U5 to U1, U3 to U10, U4 to U2, U1 to U3, U7 to U5
Connections:
- net ROUT+ is gone; now on an unnamed net: R21.2
- net ROUT- is gone; now on an unnamed net: R20.2
- net VCOM is gone; now on net +3.3V: C58.1
- net +3.3V: now also C12.1, C13.1, C33.1, C34.1, C36.1, C37.1, C39.1, C40.1, C41.1, C42.1, C43.1, C44.1, C45.1, C46.1, C48.1, C49.1, C50.1, C51.1, C54.1, C55.1, C56.1, C57.1, C59.1, C60.1, U3.105 (VDD), U3.113 (VDD), U3.120 (VDD50_USB), U3.121 (VDD33_USB), U3.126 (VDD), U3.13 (VDD), U3.135 (VDDLDO), U3.136 (VDD), U3.152 (VDD), U3.160 (VDD), U3.175 (VDDLDO), U3.176 (VDD), U3.25 (VDD), U3.44 (VDD), U3.48 (VDD), U3.65 (VDD), U3.7 (VDD), U3.71 (VDD), U3.8 (VBAT), U3.82 (VDDLDO), U3.84 (VDD), U3.92 (VDD), U3.99 (VDD), C14.1, C15.1, FB1.1, U4.7 (V_{DD}), U9.2 (VO)
- net GND: now also C53.2, R21.1, C14.2, C15.2, C16.2, C17.2, C18.2, C19.2, C26.2, C27.2, C30.2, C35.2, C38.2, C47.2, C52.2, C7.2, C8.2, C9.2, U4.16 (SGND), U4.22 (AGND2), U4.23 (AGND1), U4.28 (MODE), U4.8 (DGND), U7.1 (GND), U8.1 (PGND), U8.4 (AGND), U9.1 (GND)
- net VCC: now also C26.1, C27.1, C35.1, C38.1, U7.3 (VI), U8.2 (VIN), U8.3 (EN)
- net VDDA: now also R22.1, FB1.2; no longer L1.2
- net VGND: now also R12.1, R11.1; no longer R19.1
- net VREF+: now also R22.2, C7.1
- net at R14.2, SW4.5 (B): now also U5.6 (-)
- net at R16.1, R18.2, SW4.4 (A): now also U5.7
- net LIN_CODEC: now reaches R7.1, SW3.3 (C), U2.7
- net LIN_CODEC: now also C10.1
- net at R15.1, R17.2, SW4.1 (A): now also U5.1; no longer U5.7
- net at R20.1: now also U8.5 (FB); no longer R22.2
- net at C6.1, U3.80 (VCAP): no longer U3.133 (VCAP), U3.172 (VCAP)
- net at C53.1: now also L1.2, R19.2, C47.1, C52.1, U8.6 (VOS), U9.3 (VI)
- net at R13.2, SW4.2 (B): now also U5.2 (-); no longer U5.6 (-)
- net RIN_CODEC: now reaches R8.1, SW3.6 (C), U1.7
- net RIN_CODEC: now also C11.1
- net LOUT- renamed ROUT_CODEC
- net ROUT_CODEC: now also U4.18 (V_{OUT}R+), U5.5 (+)
- removed net VDD: C12.1, C13.1, C33.1, C34.1, C36.1, C37.1, C39.1, C40.1, C41.1, C42.1, C43.1, C44.1, C45.1, C46.1, C48.1, C49.1, C50.1, C51.1, C54.1, C55.1, C56.1, C57.1, C59.1, C60.1, L1.1, U3.105 (VDD), U3.113 (VDD), U3.120 (VDD50_USB), U3.121 (VDD33_USB), U3.126 (VDD), U3.13 (VDD), U3.135 (VDDLDO), U3.136 (VDD), U3.152 (VDD), U3.160 (VDD), U3.175 (VDDLDO), U3.176 (VDD), U3.25 (VDD), U3.44 (VDD), U3.48 (VDD), U3.65 (VDD), U3.7 (VDD), U3.71 (VDD), U3.8 (VBAT), U3.82 (VDDLDO), U3.84 (VDD), U3.92 (VDD), U3.99 (VDD)
- new net: C8.1, U3.133 (VCAP)
- new net: C9.1, U3.172 (VCAP)
- new net: L1.1, U8.7 (SW)
- new net: R19.1, U8.8 (PG)
- new net: C10.2, U4.25 (V_{IN}L)
- new net: C18.1, C19.1, U4.21 (V_{COM})
- new net: C11.2, U4.26 (V_{IN}R)
- new net +5V: C16.1, C17.1, C30.1, U4.24 (V_{CC}), U7.2 (VO)
- new net LOUT_CODEC: R11.2, U4.20 (V_{OUT}L+), U5.3 (+)
Other:
- note added: "3.8V"
- moved on the sheet: C6, J2, R6

Commit message: stuff
Parts:
- removed C38, C7: 100n, symbol Device:C
- removed SW10, SW11, SW13, SW5, SW7, SW8: SW_SP3T, symbol Switch:SW_SP3T
- removed U10: 6N139, symbol Isolator:6N139
- removed unit 2 of U6
- added C18, C19: 4.7u, symbol Device:C_Polarized
- added D2, D3: D, symbol Device:D
- added Q1, Q2: MMBT3904, Package_TO_SOT_SMD:SOT-23, symbol Transistor_BJT:MMBT3904
- added R22, R24, R26, R27: 220R, symbol Device:R
- added R23, R29, R30: 4.7K, symbol Device:R
- added R25: 1K, symbol Device:R
- added R32: 2.2K, symbol Device:R
- added R33: 10K, symbol Device:R
- added SW10, SW11, SW14, SW5, SW7, SW8: ON/OFF/ON, symbol Switch:SW_SPDT
- added U8: 6N138, symbol Isolator:6N138
- J2: value Conn_01x02_Pin -> Power in
- J7: value DIN-5_180degree -> MIDI IN
- J8: value DIN-5_180degree -> MIDI OUT
- R6: value 10K -> 220K
- RV1: value R_Potentiometer -> Pot1
- RV2: value R_Potentiometer -> Pot2
- RV3: value R_Potentiometer -> Pot3
- RV4: value R_Potentiometer -> Pot4
- RV5: value R_Potentiometer -> Pot5
- RV6: value R_Potentiometer -> Pot6
- RV7: value R_Potentiometer -> Pot7
- RV8: value R_Potentiometer -> Pot8
- U1, U2, U5, U6: value Opamp_Dual -> OPA1652
- renumbered C11 to C10, C12 to C11, C13 to C12, C14 to C13, C15 to C14, C16 to C15, C17 to C16, C18 to C17, C19 to C20, C24 to C21, C25 to C22, C20 to C23, C28 to C24, C29 to C25, C22 to C26, C31 to C27, C32 to C28, C33 to C29, C34 to C30, C36 to C31, C37 to C32, C35 to C33, C39 to C34, C40 to C35, C21 to C36, C41 to C37, C42 to C38, C23 to C39, C43 to C40, C44 to C41, C45 to C42, C46 to C43, C47 to C44, C48 to C45, C49 to C46, C50 to C47, C51 to C48, C52 to C49, C26 to C50, C54 to C51, C55 to C52, C27 to C54, C56 to C55, C57 to C56, C59 to C57, C60 to C58, C58 to C59, C30 to C60, C8 to C7, C9 to C8, C10 to C9, R12 to R10, R13 to R11, R14 to R12, R15 to R13, R16 to R14, R17 to R15, R18 to R16, R9 to R17, R10 to R18, R22 to R28, R11 to R9, U7 to U10, U8 to U7
Connections:
- net +3.3V: now also RV1.1, RV2.1, RV3.1, RV4.1, RV5.1, RV6.1, RV7.1, RV8.1, R26.2, R29.2, R30.2, R33.1, U8.8 (VCC)
- net +5V: now also K1.1, K2.1, D3.2 (A), R27.2
- net GND: now also J8.2, RV1.3, RV2.3, RV3.3, RV4.3, RV5.3, RV6.3, RV7.3, RV8.3, SW12.2, SW6.2, SW9.2, U4.27 (~{MS}/AD/IFMD), Q1.2 (E), Q2.2 (E), R25.2, SW10.2 (B), SW11.2 (B), SW14.2 (B), SW5.2 (B), SW7.2 (B), SW8.2 (B), U8.5 (GND)
- net LOUT_CODEC: now also C18.1; no longer U4.20 (V_{OUT}L+)
- net ROUT_CODEC: now also C19.1; no longer U4.18 (V_{OUT}R+)
- net POT2: now reaches RV2.2
- net POT2: now also U3.42 (PA1)
- net RELAY DRIVE: now reaches K2.16
- net RELAY DRIVE: now also K1.16, D3.1 (K), Q2.3 (C)
- net RST CODEC: now reaches U3.1 (PE2)
- net RST CODEC: now also U4.15 (~{RST}), R33.2
- net MCLK CODEC: now reaches U3.117 (PG7)
- net MCLK CODEC: now also U4.6 (SCKI1), U4.9 (SCKI2)
- net SCL CODEC: now reaches U3.165 (PB6)
- net SCL CODEC: now also U4.1 (MC/SCL/FMT), R30.1
- net SDA CODEC: now reaches U3.166 (PB7)
- net SDA CODEC: now also U4.2 (MD/SDA/DEMP), R29.1
- net TOGGLE1A: now reaches U3.18 (PF0)
- net TOGGLE1A: now also SW14.1 (A)
- net TOGGLE1B: now reaches U3.19 (PF1)
- net TOGGLE1B: now also SW14.3 (C)
- net DOUT CODEC: now reaches U3.2 (PE3)
- net DOUT CODEC: now also U4.3 (DOUT)
- net TOGGLE2A: now reaches U3.20 (PF2)
- net TOGGLE2A: now also SW5.1 (A)
- net TOGGLE2B: now reaches U3.21 (PF3)
- net TOGGLE2B: now also SW5.3 (C)
- net TOGGLE3A: now reaches U3.22 (PF4)
- net TOGGLE3A: now also SW7.1 (A)
- net TOGGLE3B: now reaches U3.23 (PF5)
- net TOGGLE3B: now also SW7.3 (C)
- net TOGGLE4A: now reaches U3.26 (PF6)
- net TOGGLE4A: now also SW8.1 (A)
- net TOGGLE4B: now reaches U3.27 (PF7)
- net TOGGLE4B: now also SW8.3 (C)
- net TOGGLE5A: now reaches U3.28 (PF8)
- net TOGGLE5A: now also SW10.1 (A)
- net TOGGLE5B: now reaches U3.29 (PF9)
- net TOGGLE5B: now also SW10.3 (C)
- net LRCK CODEC: now reaches U3.3 (PE4)
- net LRCK CODEC: now also U4.11 (LRCK2), U4.4 (LRCK1)
- net TOGGLE6A: now reaches U3.30 (PF10)
- net TOGGLE6A: now also SW11.1 (A)
- net BCK CODEC: now reaches U3.4 (PE5)
- net BCK CODEC: now also U4.10 (BCK2), U4.5 (BCK1)
- net POT1: now reaches U3.41 (PA0)
- net POT1: now also RV1.2
- net POT3: now reaches U3.43 (PA2)
- net POT3: now also RV3.2
- net POT4: now reaches U3.46 (PA3)
- net POT4: now also RV4.2
- net POT5: now reaches U3.49 (PA4)
- net POT5: now also RV5.2
- net DIN CODEC: now reaches U3.5 (PE6)
- net DIN CODEC: now also U4.12 (DIN)
- net POT6: now reaches U3.50 (PA5)
- net POT6: now also RV6.2
- net POT7: now reaches U3.51 (PA6)
- net POT7: now also RV7.2
- net POT8: now reaches U3.52 (PA7)
- net POT8: now also RV8.2
- net TOGGLE6B: now reaches U3.58 (PF11)
- net TOGGLE6B: now also SW11.3 (C)
- net FOOTSW1: now reaches U3.59 (PF12)
- net FOOTSW1: now also SW6.1
- net FOOTSW2: now reaches U3.60 (PF13)
- net FOOTSW2: now also SW9.1
- net FOOTSW3: now reaches U3.61 (PF14)
- net FOOTSW3: now also SW12.1
- net BYPASS RELAY MCU: now reaches U3.86 (PB13)
- net BYPASS RELAY MCU: now also R32.1
- net MIDI OUT MCU: now reaches U3.87 (PB14)
- net MIDI OUT MCU: now also R23.1
- net MIDI IN MCU: now reaches U3.88 (PB15)
- net MIDI IN MCU: now also R26.1, U8.6 (VO2)
- net at J7.4: now also R22.1
- net at J7.5: now also D2.2 (A), U8.3 (C2)
- net at J8.4: now also R27.1
- net at J8.5: now also R24.2
- new net: Q1.1 (B), R23.2
- new net: C18.2, U4.20 (V_{OUT}L+)
- new net: Q2.1 (B), R32.2
- new net: D2.1 (K), R22.2, U8.2 (C1)
- new net: R25.1, U8.7 (VO1)
- new net: C19.2, U4.18 (V_{OUT}R+)
- new net: Q1.3 (C), R24.1
Other:
- moved on the sheet: C10, C2, C21, C22, C23, C24, C25, C26, C27, C28, C29, C30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
