File: pcb/hopper.kicad_sch (KiCad schematic)
At the start: 141 parts, among them J1 SWD, J2 Power in, J3 L in, J4 L out, J5 R in, J6 R out, J7 MIDI IN, J8 MIDI OUT, K1 G5V-2, K2 G5V-2, Q1 MMBT3904, Q2 MMBT3904, SW1 Reset, SW10 ON/OFF/ON, SW11 ON/OFF/ON, SW12 SW_Push, SW14 ON/OFF/ON, SW2 Boot, SW3 Inst/line in, SW4 Inst/line out, SW5 ON/OFF/ON, SW6 SW_Push, SW7 ON/OFF/ON, SW8 ON/OFF/ON, SW9 SW_Push, U1 OPA1652, U10 AMS1117-5.0, U2 OPA1652, U3 STM32H745IITx, U4 PCM3060, U5 OPA1652, U6 OPA1652, U7 TPS62160DGK, U8 6N138, U9 AMS1117-3.3, Y1 Crystal_GND23

Commit message: stuff
Parts:
- removed J3: L in, symbol Connector_Audio:AudioJack2
- removed J4: L out, symbol Connector_Audio:AudioJack2
- removed J5: R in, symbol Connector_Audio:AudioJack2
- removed J6: R out, symbol Connector_Audio:AudioJack2
- added J3: L OUT, symbol Connector_Audio:AudioJack3
- added J4: R IN, symbol Connector_Audio:AudioJack3
- added J6: R OUT, symbol Connector_Audio:AudioJack3
- added J9: L IN, symbol Connector_Audio:AudioJack3
- RV1, RV8: footprint (none) -> Potentiometer_THT:Potentiometer_Alpha_RD901F-40-00D_Single_Vertical
- RV2: renamed from RV5; footprint (none) -> Potentiometer_THT:Potentiometer_Alpha_RD901F-40-00D_Single_Vertical
- RV3: renamed from RV2; footprint (none) -> Potentiometer_THT:Potentiometer_Alpha_RD901F-40-00D_Single_Vertical
- RV4: renamed from RV6; footprint (none) -> Potentiometer_THT:Potentiometer_Alpha_RD901F-40-00D_Single_Vertical
- RV5: renamed from RV3; footprint (none) -> Potentiometer_THT:Potentiometer_Alpha_RD901F-40-00D_Single_Vertical
- RV6: renamed from RV7; footprint (none) -> Potentiometer_THT:Potentiometer_Alpha_RD901F-40-00D_Single_Vertical
- RV7: renamed from RV4; footprint (none) -> Potentiometer_THT:Potentiometer_Alpha_RD901F-40-00D_Single_Vertical
- SW10: renamed from SW11; footprint (none) -> 4ms_Switch:Switch_Toggle_SPDT_Mini_SolderLug
- SW11: renamed from SW6; footprint (none) -> Connector_PinHeader_2.54mm:PinHeader_1x02_P2.54mm_Vertical
- SW12: renamed from SW9; footprint (none) -> Connector_PinHeader_2.54mm:PinHeader_1x02_P2.54mm_Vertical
- SW13: renamed from SW12; footprint (none) -> Connector_PinHeader_2.54mm:PinHeader_1x02_P2.54mm_Vertical
- SW4: renamed from SW14; footprint (none) -> 4ms_Switch:Switch_Toggle_SPDT_Mini_SolderLug
- SW5, SW7, SW8: footprint (none) -> 4ms_Switch:Switch_Toggle_SPDT_Mini_SolderLug
- SW9: renamed from SW10; footprint (none) -> 4ms_Switch:Switch_Toggle_SPDT_Mini_SolderLug
- U2, U5: footprint (none) -> Package_SO:SOIC-8-1EP_3.9x4.9mm_P1.27mm_EP2.29x3mm
- U3: renamed from U1; footprint (none) -> Package_SO:SOIC-8-1EP_3.9x4.9mm_P1.27mm_EP2.29x3mm
- U4: renamed from U6; footprint (none) -> Package_SO:SOIC-8-1EP_3.9x4.9mm_P1.27mm_EP2.29x3mm
- U9: renamed from U8; footprint (none) -> Package_DIP:DIP-8_W7.62mm
- renumbered C6 to C1, C3 to C10, C23 to C11, C26 to C12, C24 to C13, C25 to C14, C27 to C15, C28 to C16, C33 to C17, C29 to C18, C30 to C19, C7 to C2, C31 to C20, C32 to C21, C9 to C22, C10 to C23, C34 to C24, C35 to C25, C13 to C26, C14 to C27, C37 to C28, C38 to C29, C8 to C3, C44 to C30, C40 to C31, C41 to C32, C15 to C33, C49 to C34, C42 to C35, C43 to C36, C16 to C37, C17 to C38, C18 to C39, C19 to C40, C53 to C41, C20 to C42, C45 to C43, C46 to C44, C21 to C45, C22 to C46, C59 to C49, C1 to C5, C51 to C50, C52 to C51, C55 to C52, C56 to C53, C57 to C54, C58 to C55, C50 to C56, C54 to C57, C36 to C58, C39 to C59, C11 to C6, C12 to C7, C5 to C8, C2 to C9, J7 to J5, R6 to R1, R7 to R10, R8 to R11, R19 to R12, R20 to R13, R21 to R14, R9 to R15, R10 to R16, R11 to R17, R12 to R18, R13 to R19, R33 to R2, R14 to R20, R15 to R21, R16 to R22, R28 to R23, R22 to R24, R23 to R25, R32 to R26, R24 to R27, R17 to R28, R18 to R29, R25 to R30, R26 to R31, R27 to R32, R29 to R4, R30 to R5, R1 to R6, R2 to R7, R4 to R8, R5 to R9, SW4 to SW6, U3 to U1, U7 to U6, U4 to U7, U9 to U8
Connections:
- net GND: now also J3.S, J4.S, J6.S, J9.S
- net at K2.13: now also J6.T
- net at K2.4: now also J4.T
- net at K1.13: now also J3.T
- net at K1.4: now also J9.T
- no-connect marks 3 -> 7
Other:
- note added: "AUDIO"
- note added: "BYPASS"
- note added: "CODEC"
- note added: "INPUT"
- note added: "MCU"
- note added: "MIDI"
- note added: "POWER"
- moved on the sheet: C1, C10, C11, C12, C13, C14, C15, C16, C17, C18, C19, C2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
