File: pcb/hopper.kicad_sch (KiCad schematic)
At the start: 141 parts, among them J1 SWD, J2 Power in, J3 L OUT, J4 R IN, J5 MIDI IN, J6 R OUT, J8 MIDI OUT, J9 L IN, K1 G5V-2, K2 G5V-2, Q1 MMBT3904, Q2 MMBT3904, SW1 Reset, SW10 ON/OFF/ON, SW11 SW_Push, SW12 SW_Push, SW13 SW_Push, SW2 Boot, SW3 Inst/line in, SW4 ON/OFF/ON, SW5 ON/OFF/ON, SW6 Inst/line out, SW7 ON/OFF/ON, SW8 ON/OFF/ON, SW9 ON/OFF/ON, U1 STM32H745IITx, U10 AMS1117-5.0, U2 OPA1652, U3 OPA1652, U4 OPA1652, U5 OPA1652, U6 TPS62160DGK, U7 PCM3060, U8 AMS1117-3.3, U9 6N138, Y1 Crystal_GND23

Commit message: stuff
Parts:
- RV1, RV2, RV3, RV4, RV5, RV6, RV7, RV8: footprint Potentiometer_THT:Potentiometer_Alpha_RD901F-40-00D_Single_Vertical -> 4ms_Potentiometer:Pot_16mm_NoDet_RV16AF-4A
Changed lines of the file:
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@@
 			)
 		)
-		(property "Footprint" "Potentiometer_THT:Potentiometer_Alpha_RD901F-40-00D_Single_Vertical"
+		(property "Footprint" "4ms_Potentiometer:Pot_16mm_NoDet_RV16AF-4A"
 			(at 316.23 151.13 0)
 			(effects
@@
 			)
 		)
-		(property "Footprint" "Potentiometer_THT:Potentiometer_Alpha_RD901F-40-00D_Single_Vertical"
+		(property "Footprint" "4ms_Potentiometer:Pot_16mm_NoDet_RV16AF-4A"
 			(at 316.23 175.26 0)
 			(effects
@@
 			)
 		)
-		(property "Footprint" "Potentiometer_THT:Potentiometer_Alpha_RD901F-40-00D_Single_Vertical"
+		(property "Footprint" "4ms_Potentiometer:Pot_16mm_NoDet_RV16AF-4A"
 			(at 295.91 175.26 0)
 			(effects
@@
 			)
 		)
-		(property "Footprint" "Potentiometer_THT:Potentiometer_Alpha_RD901F-40-00D_Single_Vertical"
+		(property "Footprint" "4ms_Potentiometer:Pot_16mm_NoDet_RV16AF-4A"
 			(at 356.87 151.13 0)
 			(effects
@@
 			)
 		)
-		(property "Footprint" "Potentiometer_THT:Potentiometer_Alpha_RD901F-40-00D_Single_Vertical"
+		(property "Footprint" "4ms_Potentiometer:Pot_16mm_NoDet_RV16AF-4A"
 			(at 336.55 151.13 0)
 			(effects
@@
 			)
 		)
-		(property "Footprint" "Potentiometer_THT:Potentiometer_Alpha_RD901F-40-00D_Single_Vertical"
+		(property "Footprint" "4ms_Potentiometer:Pot_16mm_NoDet_RV16AF-4A"
 			(at 295.91 151.13 0)
 			(effects
@@
 			)
 		)
-		(property "Footprint" "Potentiometer_THT:Potentiometer_Alpha_RD901F-40-00D_Single_Vertical"
+		(property "Footprint" "4ms_Potentiometer:Pot_16mm_NoDet_RV16AF-4A"
 			(at 336.55 175.26 0)
 			(effects
@@
 			)
 		)
-		(property "Footprint" "Potentiometer_THT:Potentiometer_Alpha_RD901F-40-00D_Single_Vertical"
+		(property "Footprint" "4ms_Potentiometer:Pot_16mm_NoDet_RV16AF-4A"
 			(at 356.87 175.26 0)
 			(effects

Commit message: stuff
Parts:
- added J10: USB_C_Receptacle_USB2.0_16P, symbol Connector:USB_C_Receptacle_USB2.0_16P
- added R33, R34: 5.1K, symbol Device:R
- added U12: USBLC6-2SC6, Package_TO_SOT_SMD:SOT-23-6, symbol Power_Protection:USBLC6-2SC6
- Y1: value Crystal_GND23 -> 24MHz; footprint (none) -> Crystal:Crystal_SMD_3225-4Pin_3.2x2.5mm; JLC (none) -> C1122380
Connections:
- net GND: now also J10.A1 (GND), J10.A12 (GND), J10.B1 (GND), J10.B12 (GND), J10.S1 (SHIELD), R33.1, R34.1, U12.2 (GND)
- net USB DM: now reaches U1.130 (PA11)
- net USB DM: now also U12.6 (I/O1)
- net USB DP: now reaches U1.131 (PA12)
- net USB DP: now also U12.4 (I/O2)
- new net: J10.A5 (CC1), R34.2
- new net: J10.B5 (CC2), R33.2
- new net D+: J10.A6 (D+), J10.B6 (D+), U12.3 (I/O2)
- new net D-: J10.A7 (D-), J10.B7 (D-), U12.1 (I/O1)
- new net VBUS: J10.A4 (VBUS), J10.A9 (VBUS), J10.B4 (VBUS), J10.B9 (VBUS), U12.5 (VBUS)
Other:
- moved on the sheet: C1, C10, C11, C12, C13, C14, C15, C16, C17, C18, C19, C2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

Commit message: stuff
Parts:
- C5, C8: value C -> 27p
Changed lines of the file:
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@@
 			)
 		)
-		(property "Value" "C"
+		(property "Value" "27p"
 			(at 111.76 287.0199 0)
 			(effects
@@
 			)
 		)
-		(property "Value" "C"
+		(property "Value" "27p"
 			(at 91.44 287.0199 0)
 			(effects

Commit message: stuff
Parts:
- J1: footprint (none) -> Connector_PinHeader_2.54mm:PinHeader_2x05_P2.54mm_Vertical
- J3: renamed from J2; footprint (none) -> Connector_PinHeader_2.54mm:PinHeader_1x02_P2.54mm_Vertical
- J4: renamed from J9; footprint (none) -> Connector_Audio:Jack_6.35mm_Neutrik_NMJ6HCD2_Horizontal
- J5: renamed from J3; footprint (none) -> Connector_Audio:Jack_6.35mm_Neutrik_NMJ6HCD2_Horizontal
- J8: renamed from J4; footprint (none) -> Connector_Audio:Jack_6.35mm_Neutrik_NMJ6HCD2_Horizontal
- J9: renamed from J6; footprint (none) -> Connector_Audio:Jack_6.35mm_Neutrik_NMJ6HCD2_Horizontal
- renumbered J10 to J2, J5 to J6, J8 to J7, R8 to R10, R9 to R11, R10 to R12, R11 to R13, R12 to R14, R13 to R15, R14 to R16, R15 to R17, R16 to R18, R17 to R19, R18 to R20, R19 to R21, R20 to R22, R21 to R23, R22 to R24, R23 to R25, R24 to R26, R25 to R27, R26 to R28, R27 to R29, R28 to R30, R29 to R31, R30 to R32, R31 to R33, R32 to R34, R33 to R6, R34 to R7, R6 to R8, R7 to R9, U9 to U10, U10 to U11, U12 to U2, U2 to U3, U3 to U4, U4 to U5, U5 to U6, U6 to U7, U7 to U8, U8 to U9
Other:
- note added: "USB"
- moved on the sheet: J2, R6, R7, U2

Commit message: stuff
Parts:
- added C61, C62, C63, C64, C65, C66, C67, C68: 100n, Capacitor_SMD:C_0603_1608Metric, symbol Device:C
- added D4, D5, D6: APA-106-F5, LED_THT:LED_D5.0mm-4_RGB, symbol LED:APA-106-F5
- added R35: 220R, Resistor_SMD:R_0603_1608Metric, symbol Device:R
- added U12: 74AHCT125, Package_SO:SOIC-14_3.9x8.7mm_P1.27mm, symbol 74xx:74AHCT125
- C1, C10, C11, C12, C13, C14, C15, C16, C17, C18, C19, C2, C20, C21, C22, C23, C24, C25, C26, C27, C28, C29, C3, C31, C32, C33, C34, C35, C36, C37, C38, C39, C4, C40, C41, C42, C43, C44, C45, C46, C47, C48, C49, C5, C50, C51, C52, C53, C54, C55, C56, C57, C58, C59, C6, C60, C7, C8, C9: footprint (none) -> Capacitor_SMD:C_0603_1608Metric
- C30: footprint (none) -> Capacitor_SMD:C_0805_2012Metric
- D1, D2, D3: footprint (none) -> Diode_SMD:D_0603_1608Metric
- FB1, L1, R1, R10, R11, R12, R13, R14, R15, R16, R17, R18, R19, R2, R20, R21, R22, R23, R24, R25, R26, R27, R28, R29, R3, R30, R31, R32, R33, R34, R4, R5, R6, R7, R8, R9: footprint (none) -> Resistor_SMD:R_0603_1608Metric
- J2: footprint (none) -> Connector_USB:USB_C_Receptacle_GCT_USB4105-xx-A_16P_TopMnt_Horizontal
- RV1, RV2, RV3, RV4, RV5, RV6, RV7, RV8: footprint 4ms_Potentiometer:Pot_16mm_NoDet_RV16AF-4A -> 4ms_Potentiometer:Pot_9mm_DShaft
- SW1, SW2: footprint (none) -> Button_Switch_SMD:SW_SPST_TL3342
Connections:
- net +5V: now also C61.1, C62.1, C63.1, C68.1, D4.3 (VDD), D5.3 (VDD), D6.3 (VDD), U12.10, U12.13, U12.14 (VCC), U12.4
- net GND: now also C61.2, C62.2, C63.2, C64.2, C65.2, C66.2, C67.2, C68.2, D4.2 (GND), D5.2 (GND), D6.2 (GND), U12.1, U12.12, U12.5, U12.7 (GND), U12.9
- net VCC: now also C64.1, C65.1, C66.1, C67.1
- net LED DATA: now reaches U1.107 (PK0)
- net LED DATA: now also U12.2
- new net: R35.2, U12.3
- new net: D4.1 (DO), D5.4 (DI)
- new net: D4.4 (DI), R35.1
- new net: D5.1 (DO), D6.4 (DI)
- no-connect marks 7 -> 13
Other:
- note added: "LEDS"
- moved on the sheet: C11, C12, C13, C14, C15, C16, C18, C19, C20, C21, C24, C25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
