File: pcb/hopper.kicad_pcb (KiCad board)
At the start: 2 copper layers, 39 parts, among them J1 SWD, J3 Power in, J4 L IN, J5 L OUT, J8 R IN, J9 R OUT, K1 G5V-2, K2 G5V-2, Q1 MMBT3904, Q2 MMBT3904, SW10 ON/OFF/ON, SW11 SW_Push, SW12 SW_Push, SW13 SW_Push, SW4 ON/OFF/ON, SW5 ON/OFF/ON, SW7 ON/OFF/ON, SW8 ON/OFF/ON, SW9 ON/OFF/ON, U1 STM32H745IITx, U10 6N138, U11 AMS1117-5.0, U2 USBLC6-2SC6, U3 OPA1652, U4 OPA1652, U5 OPA1652, U6 OPA1652, U7 TPS62160DGK, U8 PCM3060, U9 AMS1117-3.3, Y1 24MHz

Commit message: stuff
Parts:
- added C1: 2.2u, Capacitor_SMD:C_0603_1608Metric, B.Cu at (118.4, 104.1)
- added C10: 220n, Capacitor_SMD:C_0603_1608Metric, B.Cu at (175.8, 91.4)
- added C11: 100u, Capacitor_SMD:C_0603_1608Metric, B.Cu at (6.04, -12.7)
- added C12: 100n, Capacitor_SMD:C_0603_1608Metric, B.Cu at (1.59, -42.8)
- added C13: 1u, Capacitor_SMD:C_0603_1608Metric, B.Cu at (140.0, 96.3)
- added C14: 1u, Capacitor_SMD:C_0603_1608Metric, B.Cu at (140.0, 98.0)
- added C15: 100n, Capacitor_SMD:C_0603_1608Metric, B.Cu at (140.0, 94.7)
- added C16: 100n, Capacitor_SMD:C_0603_1608Metric, B.Cu at (140.0, 99.6)
- added C17: 10u, Capacitor_SMD:C_0603_1608Metric, B.Cu at (208.9, 78.5)
- added C18: 100n, Capacitor_SMD:C_0603_1608Metric, B.Cu at (140.0, 81.0)
- added C19: 100n, Capacitor_SMD:C_0603_1608Metric, B.Cu at (109.5, 98.3)
- added C2: 2.2u, Capacitor_SMD:C_0603_1608Metric, B.Cu at (113.0, 73.7)
- added C20: 100n, Capacitor_SMD:C_0603_1608Metric, B.Cu at (140.0, 82.5)
- added C21: 100n, Capacitor_SMD:C_0603_1608Metric, B.Cu at (109.5, 94.7)
- added C22: 4.7u, Capacitor_SMD:C_0603_1608Metric, B.Cu at (151.6, 89.2)
- added C23: 4.7u, Capacitor_SMD:C_0603_1608Metric, B.Cu at (153.2, 89.2)
- added C24: 100n, Capacitor_SMD:C_0603_1608Metric, B.Cu at (140.0, 84.1)
- added C25: 100n, Capacitor_SMD:C_0603_1608Metric, B.Cu at (109.5, 91.7)
- added C26: 100n, Capacitor_SMD:C_0603_1608Metric, B.Cu at (146.8, 81.5)
- added C27: 10u, Capacitor_SMD:C_0603_1608Metric, B.Cu at (146.8, 83.1)
- added C28: 100n, Capacitor_SMD:C_0603_1608Metric, B.Cu at (140.0, 90.2)
- added C29: 100n, Capacitor_SMD:C_0603_1608Metric, B.Cu at (109.5, 87.6)
- added C3: 2.2u, Capacitor_SMD:C_0603_1608Metric, B.Cu at (132.6, 73.7)
- added C30: 22u, Capacitor_SMD:C_0805_2012Metric, B.Cu at (206.9, 83.3)
- added C31: 100n, Capacitor_SMD:C_0603_1608Metric, B.Cu at (140.0, 101.1)
- added C32: 100n, Capacitor_SMD:C_0603_1608Metric, B.Cu at (109.5, 81.0)
- added C33: 10u, Capacitor_SMD:C_0603_1608Metric, B.Cu at (158.0, 84.6)
- added C34: 10u, Capacitor_SMD:C_0603_1608Metric, B.Cu at (196.1, 81.0)
- added C35: 100n, Capacitor_SMD:C_0603_1608Metric, B.Cu at (133.9, 104.1)
- added C36: 100n, Capacitor_SMD:C_0603_1608Metric, B.Cu at (114.6, 73.7)
- added C37: 100n, Capacitor_SMD:C_0603_1608Metric, B.Cu at (158.0, 83.1)
- added C38: 10u, Capacitor_SMD:C_0603_1608Metric, B.Cu at (158.0, 80.0)
- added C39: 4.7u, Capacitor_SMD:C_0603_1608Metric, B.Cu at (151.6, 75.4)
- added C4: 100n, Capacitor_SMD:C_0603_1608Metric, B.Cu at (6.04, -33.8)
- added C40: 4.7u, Capacitor_SMD:C_0603_1608Metric, B.Cu at (153.2, 75.4)
- added C41: 100n, Capacitor_SMD:C_0603_1608Metric, B.Cu at (196.1, 78.7)
- added C42: 100n, Capacitor_SMD:C_0603_1608Metric, B.Cu at (158.0, 81.5)
- added C43: 100n, Capacitor_SMD:C_0603_1608Metric, B.Cu at (125.5, 104.1)
- added C44: 100n, Capacitor_SMD:C_0603_1608Metric, B.Cu at (116.1, 73.7)
- added C45: 10u, Capacitor_SMD:C_0603_1608Metric, B.Cu at (178.3, 83.6)
- added C46: 10u, Capacitor_SMD:C_0603_1608Metric, B.Cu at (165.1, 79.8)
- added C47: 100n, Capacitor_SMD:C_0603_1608Metric, B.Cu at (122.4, 104.1)
- added C48: 100n, Capacitor_SMD:C_0603_1608Metric, B.Cu at (123.4, 73.7)
- added C49: 10u, Capacitor_SMD:C_0603_1608Metric, B.Cu at (183.9, 77.0)
- added C5: 27p, Capacitor_SMD:C_0603_1608Metric, B.Cu at (145.7, 91.0)
- added C50: 100n, Capacitor_SMD:C_0603_1608Metric, B.Cu at (116.8, 104.1)
- added C51: 100n, Capacitor_SMD:C_0603_1608Metric, B.Cu at (127.5, 73.7)
- added C52: 100n, Capacitor_SMD:C_0603_1608Metric, B.Cu at (115.3, 104.1)
- added C53: 100n, Capacitor_SMD:C_0603_1608Metric, B.Cu at (135.6, 73.7)
- added C54: 4.7u, Capacitor_SMD:C_0603_1608Metric, B.Cu at (138.7, 73.7)
- added C55: 100n, Capacitor_SMD:C_0603_1608Metric, B.Cu at (137.2, 73.7)
- added C56: 10u, Capacitor_SMD:C_0603_1608Metric, B.Cu at (181.6, 59.2)
- added C57: 100n, Capacitor_SMD:C_0603_1608Metric, B.Cu at (179.1, 59.2)
- added C58: 10u, Capacitor_SMD:C_0603_1608Metric, B.Cu at (-16.2, -36.8)
- added C59: 100n, Capacitor_SMD:C_0603_1608Metric, B.Cu at (-16.2, -33.8)
- added C6: 100n, Capacitor_SMD:C_0603_1608Metric, B.Cu at (109.5, 83.1)
- added C60: 10u, Capacitor_SMD:C_0603_1608Metric, B.Cu at (177.0, 71.4)
- added C61: 100n, Capacitor_SMD:C_0603_1608Metric, B.Cu at (104.1, 108.0)
- added C62: 100n, Capacitor_SMD:C_0603_1608Metric, B.Cu at (152.4, 108.0)
- added C63: 100n, Capacitor_SMD:C_0603_1608Metric, B.Cu at (200.7, 108.0)
- added C64: 100n, Capacitor_SMD:C_0603_1608Metric, B.Cu at (170.4, 94.2)
- added C65: 100n, Capacitor_SMD:C_0603_1608Metric, B.Cu at (170.4, 87.1)
- added C66: 100n, Capacitor_SMD:C_0603_1608Metric, B.Cu at (27.9, 43.4)
- added C67: 100n, Capacitor_SMD:C_0603_1608Metric, B.Cu at (170.4, 80.0)
- added C68: 100n, Capacitor_SMD:C_0603_1608Metric, B.Cu at (27.9, 48.4)
- added C7: 1u, Capacitor_SMD:C_0603_1608Metric, B.Cu at (109.5, 84.6)
- added C8: 27p, Capacitor_SMD:C_0603_1608Metric, B.Cu at (145.7, 96.6)
- added C9: 220n, Capacitor_SMD:C_0603_1608Metric, B.Cu at (175.8, 98.6)
- added D1: D_Schottky, Diode_SMD:D_0603_1608Metric, B.Cu at (59.3, -31.2)
- added D2: D, Diode_SMD:D_0603_1608Metric, B.Cu at (59.3, -28.1)
- added D3: D, Diode_SMD:D_0603_1608Metric, B.Cu at (208.3, 108.2)
- added D4: APA-106-F5, LED_THT:LED_D5.0mm-4_RGB, F.Cu at (102.2, 111.8)
- added D5: APA-106-F5, LED_THT:LED_D5.0mm-4_RGB, F.Cu at (150.5, 111.8)
- added D6: APA-106-F5, LED_THT:LED_D5.0mm-4_RGB, F.Cu at (198.8, 111.8)
- added FB1: FerriteBead_Small, Resistor_SMD:R_0603_1608Metric, B.Cu at (142.2, 98.8)
- added J2: USB_C_Receptacle_USB2.0_16P, Connector_USB:USB_C_Receptacle_GCT_USB4105-xx-A_16P_TopMnt_Horizontal, B.Cu at (274.6, -14.5)
- added L1: 2.2uH, Resistor_SMD:R_0603_1608Metric, B.Cu at (200.3, 78.5)
- added R1: 220K, Resistor_SMD:R_0603_1608Metric, B.Cu at (134.1, 73.7)
- added R10: 10K, Resistor_SMD:R_0603_1608Metric, B.Cu at (165.1, 91.4)
- added R11: 10K, Resistor_SMD:R_0603_1608Metric, B.Cu at (165.1, 98.6)
- added R12: 30.1K, Resistor_SMD:R_0603_1608Metric, B.Cu at (165.1, 97.0)
- added R13: 30.1K, Resistor_SMD:R_0603_1608Metric, B.Cu at (165.1, 89.9)
- added R14: 100K, Resistor_SMD:R_0603_1608Metric, B.Cu at (204.6, 75.2)
- added R15: 220K, Resistor_SMD:R_0603_1608Metric, B.Cu at (203.3, 81.3)
- added R16: 100K, Resistor_SMD:R_0603_1608Metric, B.Cu at (206.9, 81.3)
- added R17: 100K, Resistor_SMD:R_0603_1608Metric, B.Cu at (175.8, 85.9)
- added R18: 100K, Resistor_SMD:R_0603_1608Metric, B.Cu at (165.1, 85.9)
- added R19: 10K, Resistor_SMD:R_0603_1608Metric, B.Cu at (175.8, 84.3)
- added R2: 10K, Resistor_SMD:R_0603_1608Metric, B.Cu at (140.0, 77.0)
- added R20: 10K, Resistor_SMD:R_0603_1608Metric, B.Cu at (165.1, 84.3)
- added R21: 10K, Resistor_SMD:R_0603_1608Metric, B.Cu at (175.8, 82.8)
- added R22: 10K, Resistor_SMD:R_0603_1608Metric, B.Cu at (165.1, 82.8)
- added R23: 100R, Resistor_SMD:R_0603_1608Metric, B.Cu at (175.8, 81.3)
- added R24: 100R, Resistor_SMD:R_0603_1608Metric, B.Cu at (165.1, 81.3)
- added R25: 47R, Resistor_SMD:R_0603_1608Metric, B.Cu at (142.2, 95.5)
- added R26: 220R, Resistor_SMD:R_0603_1608Metric, B.Cu at (63.8, -31.2)
- added R27: 4.7K, Resistor_SMD:R_0603_1608Metric, B.Cu at (63.8, -28.3)
- added R28: 2.2K, Resistor_SMD:R_0603_1608Metric, B.Cu at (63.8, -25.3)
- added R29: 220R, Resistor_SMD:R_0603_1608Metric, B.Cu at (63.8, -22.4)
- added R3: 10K, Resistor_SMD:R_0603_1608Metric, B.Cu at (77.0, -19.4)
- added R30: 47K, Resistor_SMD:R_0603_1608Metric, B.Cu at (63.8, -19.4)
- added R31: 47K, Resistor_SMD:R_0603_1608Metric, B.Cu at (63.8, -16.5)
- added R32: 1K, Resistor_SMD:R_0603_1608Metric, B.Cu at (63.8, -13.5)
- added R33: 220R, Resistor_SMD:R_0603_1608Metric, B.Cu at (63.8, -10.6)
- added R34: 220R, Resistor_SMD:R_0603_1608Metric, B.Cu at (63.8, -7.62)
- added R35: 220R, Resistor_SMD:R_0603_1608Metric, B.Cu at (27.9, 50.9)
- added R4: 4.7K, Resistor_SMD:R_0603_1608Metric, B.Cu at (131.1, 73.7)
- added R5: 4.7K, Resistor_SMD:R_0603_1608Metric, B.Cu at (129.5, 73.7)
- added R6: 5.1K, Resistor_SMD:R_0603_1608Metric, B.Cu at (77.0, -10.6)
- added R7: 5.1K, Resistor_SMD:R_0603_1608Metric, B.Cu at (77.0, -7.62)
- added R8: 1M, Resistor_SMD:R_0603_1608Metric, B.Cu at (175.8, 97.0)
- added R9: 1M, Resistor_SMD:R_0603_1608Metric, B.Cu at (175.8, 89.9)
- added SW1: Reset, Button_Switch_SMD:SW_SPST_TL3342, B.Cu at (264.0, -16.3)
- added SW2: Boot, Button_Switch_SMD:SW_SPST_TL3342, B.Cu at (264.0, -9.25)
- added U12: 74AHCT125, Package_SO:SOIC-14_3.9x8.7mm_P1.27mm, B.Cu at (101.6, 97.8)
- J1, J3, K1, K2, Q1, Q2, SW11, SW12, SW13, U1, U10, U11, U2, U3, U4, U5, U6, U7, U8, U9, Y1: moved to B.Cu
- RV1, RV2, RV3, RV4, RV5, RV6, RV7, RV8: footprint 4ms_Potentiometer:Pot_16mm_NoDet_RV16AF-4A -> 4ms_Potentiometer:Pot_9mm_DShaft
- moved SW13 239.3 mm to (113.0, 111.8), turned to -90 degrees
- moved U1 228.4 mm to (124.7, 88.9), turned to 180 degrees
- moved SW12 213.8 mm to (141.0, 111.8), turned to -90 degrees
- moved J1 206.5 mm to (102.9, 76.2), turned to 180 degrees
- moved U8 202.8 mm to (152.4, 82.3)
- moved Y1 188.9 mm to (145.7, 93.8)
- moved SW11 177.2 mm to (189.2, 111.8), turned to -90 degrees
- moved U10 170.3 mm to (141.0, -24.1), turned to 180 degrees
- moved Q2 167.9 mm to (208.3, 111.5), turned to 90 degrees
- moved U3 157.7 mm to (170.4, 97.8), turned to 180 degrees
- moved K1 154.6 mm to (202.4, 104.3), turned to 90 degrees
- moved K2 148.8 mm to (202.4, 93.5), turned to 90 degrees
- moved U7 148.6 mm to (204.6, 78.5), turned to 180 degrees
- moved U9 148.0 mm to (189.7, 78.7), turned to 180 degrees
- moved U4 145.8 mm to (170.4, 90.7), turned to 180 degrees
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Connections:
- U1 pad 107: unconnected-(U1-PK0-Pad107) -> LED DATA
Routing:
- net MCLK CODEC: track 0.00 -> 49.9 mm, vias 0 -> 2
- net +3.3V: track 0.00 -> 49.8 mm, vias 0 -> 31
- net LOUT_CODEC: track 0.00 -> 31.2 mm, vias 0 -> 2
- net LRCK CODEC: track 0.00 -> 25.9 mm, vias 0 -> 2
- net DOUT CODEC: track 0.00 -> 24.4 mm
- net VCC: track 0.00 -> 23.9 mm, vias 0 -> 3
- net BCK CODEC: track 0.00 -> 22.2 mm, vias 0 -> 2
- net ROUT: track 0.00 -> 21.8 mm
- net VGND: track 0.00 -> 21.1 mm
- net ROUT_CODEC: track 0.00 -> 19.6 mm, vias 0 -> 2
- net LIN_CODEC: track 0.00 -> 19.3 mm, vias 0 -> 2
- net LOUT: track 0.00 -> 15.9 mm
- net RIN_CODEC: track 0.00 -> 14.9 mm, vias 0 -> 2
- net DIN CODEC: track 0.00 -> 12.5 mm
- net LIN: track 0.00 -> 10.5 mm
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- added copper zone on In2.Cu, net +3.3V
- added copper zone on B.Cu, net GND
- added copper zone on F.Cu, net GND
- added copper zone on In1.Cu, net GND
Other:
- board outline added: 119.4 x 83.8 mm
- copper layers 2 -> 4
- board text added: "${REFERENCE}"
