File: hardware/hopper.kicad_sch (KiCad schematic)
At the start: 170 parts, among them J1 SWD, J2 USB_C_Receptacle_USB2.0_16P, J3 Power in, J4 L IN, J5 L OUT, J6 MIDI IN, J7 MIDI OUT, J8 R IN, J9 R OUT, K1 G5V-2, K2 G5V-2, Q1 MMBT3904, Q2 MMBT3904, SW1 Reset, SW10 ON/OFF/ON, SW11 FS1, SW12 FS2, SW13 FS3, SW2 Boot, SW3 Inst/line in, SW4 ON/OFF/ON, SW5 ON/OFF/ON, SW6 Inst/line out, SW7 ON/OFF/ON, SW8 ON/OFF/ON, SW9 ON/OFF/ON, U1 STM32H745IITx, U10 6N138, U11 AMS1117-5.0, U12 74AHCT125, U13 STM32H750VBTx, U2 USBLC6-2SC6, U3 OPA1652, U4 OPA1652, U5 OPA1652, U6 OPA1652, U7 TPS62160DGK, U8 PCM3060, U9 AMS1117-3.3, Y1 24MHz

Commit message: Add ADC1 channel configuration and GPIO pin assignments to STM32 IOC
Parts:
- U3, U4, U5, U6: value OPA1652 -> OPA1642
Connections:
- net BYPASS RELAY MCU: now also U13.90 (PB4); no longer U13.34 (PB0)
- net LED DATA: now also U13.63 (PC6); no longer U13.15 (PC0)
- net MIDI IN MCU: now also U13.92 (PB6); no longer U13.36 (PB2)
- net MIDI OUT MCU: now also U13.91 (PB5); no longer U13.35 (PB1)
- net POT1: now also U13.22 (PA0); no longer U13.81 (PD0)
- net POT2: now also U13.23 (PA1); no longer U13.82 (PD1)
- net POT3: now also U13.24 (PA2); no longer U13.83 (PD2)
- net POT4: now also U13.25 (PA3); no longer U13.84 (PD3)
- net POT5: now also U13.28 (PA4); no longer U13.85 (PD4)
- net POT6: now also U13.29 (PA5); no longer U13.86 (PD5)
- net POT7: now also U13.30 (PA6); no longer U13.87 (PD6)
- net POT8: now also U13.31 (PA7); no longer U13.88 (PD7)
- net TOGGLE1: now also U13.32 (PC4); no longer U13.46 (PB10)
- net TOGGLE2: now also U13.33 (PC5); no longer U13.47 (PB11)
- net TOGGLE3: now also U13.15 (PC0); no longer U13.51 (PB12)
- net TOGGLE4: now also U13.16 (PC1); no longer U13.52 (PB13)
- net TOGGLE5: now also U13.34 (PB0); no longer U13.53 (PB14)
- net TOGGLE6: now also U13.35 (PB1); no longer U13.54 (PB15)
Other:
- moved on the sheet: C5, C69, C70, C8, J1, R36, R37, R38, U13, Y1

Commit message: Add I2C4 peripheral, configure ADC pull-downs, and update PLL2 clocks
Parts:
- removed C1, C2, C3: 2.2u, Capacitor_SMD:C_0603_1608Metric, symbol Device:C
- removed R2: 10K, Resistor_SMD:R_0603_1608Metric, symbol Device:R
- removed R4, R5: 4.7K, Resistor_SMD:R_0603_1608Metric, symbol Device:R
- removed U13: STM32H750VBTx, Package_QFP:LQFP-100_14x14mm_P0.5mm, symbol MCU_ST_STM32H7:STM32H750VBTx
- added U13: STM32H743VITx, Package_QFP:LQFP-100_14x14mm_P0.5mm, symbol MCU_ST_STM32H7:STM32H743VITx
Connections:
- net +3.3V: now also U13.100 (VDD), U13.11 (VDD), U13.27 (VDD), U13.50 (VDD), U13.6 (VBAT), U13.75 (VDD)
- net BCK CODEC: now also U13.4 (PE5); no longer U1.4 (PE5)
- net BOOT: now also U13.94 (BOOT0); no longer U1.167 (BOOT0)
- net BYPASS RELAY MCU: now also U13.90 (PB4); no longer U1.86 (PB13)
- net CRYSTAL1: now also U13.12 (PH0); no longer U1.31 (PH0)
- net CRYSTAL2: now also U13.13 (PH1); no longer U1.32 (PH1)
- net DIN CODEC: now also U13.5 (PE6); no longer U1.5 (PE6)
- net DOUT CODEC: now also U13.2 (PE3); no longer U1.2 (PE3)
- net FOOTSW1: now also U13.7 (PC13); no longer U1.59 (PF12)
- net FOOTSW2: now also U13.8 (PC14); no longer U1.60 (PF13)
- net FOOTSW3: now also U13.9 (PC15); no longer U1.61 (PF14)
- net GND: now also U13.10 (VSS), U13.19 (VSSA), U13.26 (VSS), U13.49 (VSS), U13.74 (VSS), U13.99 (VSS)
- net LED DATA: now also U13.63 (PC6); no longer U1.107 (PK0)
- net LRCK CODEC: now also U13.3 (PE4); no longer U1.3 (PE4)
- net MCLK CODEC: now also U13.1 (PE2); no longer U1.117 (PG7)
- net MIDI IN MCU: now also U13.92 (PB6); no longer U1.88 (PB15)
- net MIDI OUT MCU: now also U13.91 (PB5); no longer U1.87 (PB14)
- net POT1: now also U13.22 (PA0); no longer U1.41 (PA0)
- net POT2: now also U13.23 (PA1); no longer U1.42 (PA1)
- net POT3: now also U13.24 (PA2); no longer U1.43 (PA2)
- net POT4: now also U13.25 (PA3); no longer U1.46 (PA3)
- net POT5: now also U13.28 (PA4); no longer U1.49 (PA4)
- net POT6: now also U13.29 (PA5); no longer U1.50 (PA5)
- net POT7: now also U13.30 (PA6); no longer U1.51 (PA6)
- net POT8: now also U13.31 (PA7); no longer U1.52 (PA7)
- net RST: now also U13.14 (NRST); no longer U1.33 (NRST)
- net RST CODEC: now also U13.98 (PE1); no longer U1.1 (PE2)
- net SCL CODEC: now also R37.1, U13.59 (PD12); no longer R36.1, U1.165 (PB6)
- net SDA CODEC: now also R36.1, U13.60 (PD13); no longer R37.1, U1.166 (PB7)
- net SWCLK: now also U13.76 (PA14); no longer U1.138 (PA14)
- net SWDIO: now also U13.72 (PA13); no longer U1.132 (PA13)
- net SWO: now also U13.89 (PB3); no longer U1.162 (PB3)
- net TOGGLE1: now also U13.32 (PC4)
- net TOGGLE2: now also U13.33 (PC5)
- net TOGGLE3: now also U13.15 (PC0)
- net TOGGLE4: now also U13.16 (PC1)
- net TOGGLE5: now also U13.34 (PB0)
- net TOGGLE6: now also U13.35 (PB1)
- net USB DM: now also U13.70 (PA11); no longer U1.130 (PA11)
- net USB DP: now also U13.71 (PA12); no longer U1.131 (PA12)
- net VDDA: now also U13.21 (VDDA)
- net VREF+: now also U13.20 (VREF+); no longer U1.39 (VREF+)
- net at C69.1: now also U13.48 (VCAP)
- net at C70.1: now also U13.73 (VCAP)
- net TOGGLE1A: no longer names the net of U1.18 (PF0)
- net TOGGLE1B: no longer names the net of U1.19 (PF1)
- net TOGGLE2A: no longer names the net of U1.20 (PF2)
- net TOGGLE2B: no longer names the net of U1.21 (PF3)
- net TOGGLE3A: no longer names the net of U1.22 (PF4)
- net TOGGLE3B: no longer names the net of U1.23 (PF5)
- net TOGGLE4A: no longer names the net of U1.26 (PF6)
- net TOGGLE4B: no longer names the net of U1.27 (PF7)
- net TOGGLE5A: no longer names the net of U1.28 (PF8)
- net TOGGLE5B: no longer names the net of U1.29 (PF9)
- net TOGGLE6A: no longer names the net of U1.30 (PF10)
- net TOGGLE6B: no longer names the net of U1.58 (PF11)
Other:
- note added: "Connected to ADC1"
- note added: "Connected to ADC1 with pull-downs enabled"
- moved on the sheet: R39, R40, R41, R42, R43, R44, RV1, RV2, RV3, RV4, RV5, RV6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

Commit message: Add STM32CubeMX-generated firmware sources, HAL drivers, and CMake build system
Parts:
- removed C19, C21, C25, C29, C32, C35, C36, C43, C44, C47, C48, C50, C51, C52, C53, C55, C6: 100n, Capacitor_SMD:C_0603_1608Metric, symbol Device:C
- removed C7: 1u, Capacitor_SMD:C_0603_1608Metric, symbol Device:C_Polarized
- removed J3: Power in, Connector_PinHeader_2.54mm:PinHeader_1x02_P2.54mm_Vertical, symbol Connector:Conn_01x02_Pin
- removed R1: 220K, Resistor_SMD:R_0603_1608Metric, symbol Device:R
- removed U1: STM32H745IITx, Package_QFP:LQFP-176_24x24mm_P0.5mm, symbol MCU_ST_STM32H7:STM32H745IITx
- added J10: 9V, symbol Connector:Barrel_Jack_Switch
- added J3: Micro_SD_Card, symbol Connector:Micro_SD_Card
Connections:
- net +9V: now also J10.2
- net GND: now also J10.1
Other:
- note removed: "Near usb power pins"
- moved on the sheet: C11, C12, C13, C14, C15, C16, C18, C20, C24, C28, C31, C4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
